File: hardware_PicoKey/hardware_PicoKey.kicad_pcb (KiCad board)
At the start: 2 copper layers, 36.9 x 18.5 mm, 36 parts, among them J1 USB_A, SW1 SW_Push, SW2 SW_Push, U1 RP2350A-QFN60, U2 AMS1117S-3.3, U3 W25Q128JVS, Y1 Crystal_GND24

Commit message: pcb
Parts:
- C1, C18, C19, C2, C3, R1, R4, R5: moved to B.Cu
- moved C2 32.5 mm to (136.2, 71.8), turned to 90 degrees
- moved C3 30.4 mm to (137.8, 71.2), turned to -90 degrees
- moved C1 30.4 mm to (139.7, 73.0)
- moved R1 29.3 mm to (137.2, 73.2)
- moved C18 20.4 mm to (153.5, 71.9)
- moved C19 19.4 mm to (153.8, 66.7), turned to 180 degrees
- moved R5 13.5 mm to (151.0, 70.0), turned to 180 degrees
- moved Y1 11.4 mm to (153.8, 69.2), turned to -90 degrees
- moved L1 10.6 mm to (138.8, 71.2), turned to 90 degrees
- moved D2 9.05 mm to (144.8, 62.5), turned to 0 degrees
- moved U3 8.65 mm to (139.2, 64.5), turned to -90 degrees
- moved SW1 7.77 mm to (150.0, 64.8)
- moved C4 6.77 mm to (138.0, 75.2), turned to -90 degrees
- moved C10 6.68 mm to (164.0, 64.6)
- moved C11 6.68 mm to (164.0, 66.6)
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Connections:
- D2 pad 1: USB_DP -> USB_DM
- D2 pad 2: unconnected-(D2-GND-Pad2) -> GND
- D2 pad 3: USB_DM -> USB_DP
Routing:
- net USB_DP: track 0.00 -> 22.1 mm, vias 0 -> 2
- net USB_DM: track 0.00 -> 21.9 mm, vias 0 -> 2
- net QSPI_SD2: track 0.00 -> 8.87 mm, vias 0 -> 1
- net QSPI_SD1: track 0.00 -> 7.30 mm, vias 0 -> 1
- net QSPI_SS: track 0.00 -> 5.69 mm, vias 0 -> 1
- net Net-(U1-USB_DP): track 0.00 -> 5.28 mm
- net QSPI_SD0: track 0.00 -> 5.07 mm, vias 0 -> 1
- net Net-(U1-USB_DM): track 0.00 -> 5.03 mm
- net QSPI_SCLK: track 0.00 -> 4.59 mm, vias 0 -> 1
- net 1v1: track 0.00 -> 4.32 mm
- net Net-(U1-VREG_LX): track 0.00 -> 3.38 mm
- net QSPI_SD3: track 0.00 -> 2.97 mm, vias 0 -> 1

Commit message: 'pcb'
Parts:
- C6, C7, C8: moved to B.Cu
- moved C8 15.9 mm to (145.5, 75.2), turned to -90 degrees
- moved C6 15.4 mm to (147.5, 61.2), turned to 90 degrees
- moved C7 10.6 mm to (150.5, 70.2), turned to -90 degrees
- moved C10 7.36 mm to (171.3, 65.6)
- moved C11 7.36 mm to (171.3, 67.6)
- moved C12 7.36 mm to (171.3, 69.6)
- moved C13 7.36 mm to (171.3, 71.5)
- moved C14 7.36 mm to (171.3, 73.5)
- moved C9 7.36 mm to (171.3, 63.6)
- moved C15 7.36 mm to (174.1, 63.6)
- moved C16 7.36 mm to (174.1, 65.6)
- moved C17 7.36 mm to (174.1, 67.6)
- moved R5 0.71 mm to (151.5, 70.5), turned to 90 degrees
- moved C19 0.40 mm to (153.8, 66.2)
- moved Y1 0.40 mm to (153.8, 68.8)
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Routing:
- net 1v1: track 4.32 -> 10.2 mm
- net Net-(U1-VREG_AVDD): track 0.00 -> 3.08 mm

Commit message: pcb
Parts:
- C11, C12, C13, C14, C15, C16, C17: moved to B.Cu
- moved C9 35.6 mm to (136.2, 70.2)
- moved C10 35.5 mm to (136.2, 71.2)
- moved C16 32.1 mm to (143.5, 75.2), turned to -90 degrees
- moved C15 31.4 mm to (142.8, 63.5), turned to 90 degrees
- moved C17 27.0 mm to (148.2, 75.2), turned to -90 degrees
- moved C11 26.8 mm to (144.8, 63.5), turned to 90 degrees
- moved C12 20.5 mm to (151.0, 66.8)
- moved C13 20.1 mm to (151.2, 73.0)
- moved C14 20.1 mm to (151.2, 72.0)
- moved R6 18.3 mm to (145.5, 61.5), turned to 180 degrees
- moved D2 5.25 mm to (150.0, 62.5)
- moved R2 3.35 mm to (147.8, 67.5)
- moved R7 3.01 mm to (147.2, 71.8)
- moved C6 2.85 mm to (145.8, 63.5)
- moved C5 2.00 mm to (141.8, 75.5)
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Connections:
- R7 pad 1: Net-(U1-GPIO11) -> Net-(U1-GPIO25)
- U1 pad 15: Net-(U1-GPIO11) -> unconnected-(U1-GPIO11-Pad15)
- U1 pad 37: unconnected-(U1-GPIO25-Pad37) -> Net-(U1-GPIO25)
Routing:
- net 3v3: track 0.00 -> 73.9 mm, vias 0 -> 3
- net Net-(R6-Pad1): track 0.00 -> 7.12 mm
- net Net-(U1-USB_DP): track 5.28 -> 0.01 mm
- net Net-(U1-USB_DM): track 5.03 -> 0.24 mm
- net QSPI_SS: track 5.69 -> 9.76 mm
- net USB_DM: track 21.9 -> 24.6 mm
- net Net-(U1-GPIO8): track 0.00 -> 2.08 mm, vias 0 -> 1
- net USB_DP: track 22.1 -> 23.7 mm
- net 1v1: track 10.2 -> 8.65 mm
- net QSPI_SCLK: track 4.59 -> 3.36 mm
- net QSPI_SD0: track 5.07 -> 6.07 mm
Other:
- board size 36.9 x 18.5 mm -> 37 x 18.5 mm

Commit message: 'pcb'
Routing:
- net USB_DM: track 24.6 -> 28.5 mm
- net USB_DP: track 23.7 -> 27.5 mm
Changed lines of the file:
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@@
+	)
+	(segment
+		(start 133.29994 68.75)
+		(end 135.99 68.75)
+		(width 0.2)
+		(layer "B.Cu")
+		(net 9)
+	)
+	(segment
+		(start 132.54994 68)
+		(end 133.29994 68.75)
+		(width 0.2)
+		(layer "B.Cu")
+		(net 9)
 	)
 	(segment
 		(start 142.5 61.5125)
 		(end 142.5875 61.6)
+		(width 0.2)
+		(layer "B.Cu")
+		(net 9)
+	)
+	(segment
+		(start 132.5 68)
+		(end 132.54994 68)
 		(width 0.2)
 		(layer "B.Cu")
@@
 	)
 	(segment
+		(start 133.449997 69.75)
+		(end 135.99 69.75)
+		(width 0.2)
+		(layer "B.Cu")
+		(net 10)
+	)
+	(segment
 		(start 132.54994 68.800003)
 		(end 132.5 68.800003)
 		(width 0.2)
 		(layer "B.Cu")
+		(net 10)
+	)
+	(segment
+		(start 132.5 68.800003)
+		(end 133.449997 69.75)
+		(width 0.2)
+		(layer "B.Cu")

Commit message: pcb and journaling
Parts:
- C10, C9: moved to B.Cu
- moved C10 8.34 mm to (137.5, 63.0)
- moved C9 6.37 mm to (137.5, 64.0)
- moved D1 3.14 mm to (149.9, 69.6)
- moved R2 2.10 mm to (147.7, 69.6)
- moved R7 1.27 mm to (146.0, 72.0)
Routing:
- net Net-(U1-USB_DP): track 0.01 -> 5.18 mm
- net Net-(U1-USB_DM): track 0.24 -> 5.17 mm
- net USB_DM: track 28.5 -> 23.9 mm
- net USB_DP: track 27.5 -> 23.9 mm
- net Net-(U1-GPIO8): track 2.08 -> 4.20 mm
- net Net-(D1-A): track 0.00 -> 1.21 mm
Other:
- board size 37 x 18.5 mm -> 34.5 x 18.5 mm

Commit message: pcb
Parts:
- D1: footprint LED_SMD:LED_0402_1005Metric -> LED_SMD:LED_0402_1005Metric_Pad0.77x0.64mm_HandSolder
- R2, R6, R7: footprint Resistor_SMD:R_0402_1005Metric -> Resistor_SMD:R_0402_1005Metric_Pad0.72x0.64mm_HandSolder
- moved D1 1.63 mm to (151.5, 69.6)
- moved C8 0.75 mm to (144.8, 75.2)
- moved R2 0.57 mm to (148.3, 69.6)
- moved C11 0.50 mm to (144.2, 63.5)
- moved C14 0.25 mm to (151.2, 72.2)
- moved C19 0.25 mm to (153.8, 66.0)
- moved C4 0.25 mm to (138.0, 75.5)
- moved C13 0.22 mm to (151.2, 73.2)
Routing:
- net GND: track 0.00 -> 70.0 mm, vias 0 -> 12
- net 3v3: track 73.9 -> 99.4 mm, vias 3 -> 5
- net 1v1: track 8.65 -> 32.0 mm, vias 0 -> 3
- net Net-(J1-VBUS): track 0.00 -> 17.1 mm, vias 0 -> 1
- net XIN: track 0.00 -> 8.10 mm
- net Net-(R7-Pad2): track 0.00 -> 6.12 mm
- net USB_DM: track 23.9 -> 28.7 mm
- net USB_DP: track 23.9 -> 28.7 mm
- net Net-(U1-GPIO25): track 0.00 -> 4.54 mm, vias 0 -> 1
- net Net-(C18-Pad1): track 0.00 -> 3.80 mm
- net XOUT: track 0.00 -> 3.57 mm
- net Net-(U1-VREG_AVDD): track 3.08 -> 5.57 mm
- net Net-(D1-A): track 1.21 -> 2.09 mm
- added copper zone on B.Cu, net GND
- added copper zone on F.Cu, net GND

Commit message: pcb donee
Parts:
- added G***: LOGO, LOGO, F.Cu at (155.0, 68.5)
- moved SW2 2.30 mm to (150.0, 72.2)
- moved D1 1.12 mm to (151.5, 68.5)
- moved R2 1.10 mm to (148.2, 68.5)
Routing:
- net GND: track 70.0 -> 104.3 mm
- net Net-(U1-GPIO8): track 4.44 -> 3.35 mm
- net Net-(R6-Pad1): track 7.12 -> 7.76 mm
Other:
- board text added: "Made By Keyaan!"

Commit message: PCB
Parts:
- L1: footprint Inductor_SMD:L_0402_1005Metric -> Inductor_SMD:L_0805_2012Metric
- moved C1 2.50 mm to (139.8, 75.5)
- moved L1 1.78 mm to (139.2, 72.9)
- moved C4 1.25 mm to (137.2, 76.5)
- moved C5 1.03 mm to (142.0, 76.5)
- moved C10 1.00 mm to (137.5, 64.0)
- moved C11 1.00 mm to (144.2, 64.5)
- moved C12 1.00 mm to (151.0, 67.8)
- moved C13 1.00 mm to (151.2, 74.2)
- moved C14 1.00 mm to (151.2, 73.2)
- moved C15 1.00 mm to (142.8, 64.5)
- moved C16 1.00 mm to (143.5, 76.2)
- moved C17 1.00 mm to (148.2, 76.2)
- moved C18 1.00 mm to (153.8, 72.8)
- moved C19 1.00 mm to (153.8, 67.0)
- moved C2 1.00 mm to (136.2, 72.8)
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Routing:
- net GND: track 104.3 -> 112.8 mm, vias 12 -> 13
- net Net-(U1-VREG_AVDD): track 5.57 -> 7.47 mm
- net 3v3: track 99.4 -> 100.8 mm
- net Net-(J1-VBUS): track 17.1 -> 16.4 mm
