File: hardware_PicoKey/hardware_PicoKey.kicad_pcb (KiCad board)
At the start: 2 copper layers, 34.5 x 18.5 mm, 37 parts, among them J1 USB_A, SW1 SW_Push, SW2 SW_Push, U1 RP2350A-QFN60, U2 AMS1117S-3.3, U3 W25Q128JVS, Y1 Crystal_GND24

Commit message: pcb
Other:
- board text added: "BOOT"
- board text added: "HACK!"
- board text added: "OPEN SOURCE!"
- board text added: "github.com/Keyaan-07/PicoKey"
- board text added: "😃"
