File: hardware_PicoKey/hardware_PicoKey.kicad_sch (KiCad schematic)
At the start: 0 parts

Commit message: schematic
Parts:
- added C1, C2, C3: 4.7u, symbol Device:C
- added C10, C11, C12, C13, C14, C15, C16, C17, C6, C7, C8, C9: 100n, symbol Device:C
- added C4, C5: 10u, symbol Device:C
- added D1: LED, symbol Device:LED
- added J1: USB_A, symbol Connector:USB_A
- added L1: 3.3u, symbol Device:L
- added R1, R2: 33, symbol Device:R
- added R3, R4: 27, symbol Device:R
- added U1: RP2350A-QFN60, user_imported_devices:RP2350A_QFN-60_EP_7.75x7.75_Pitch0.4mm, symbol user_imported:RP2350A-QFN60
- added U2: AMS1117S-3.3, Package_TO_SOT_SMD:SOT-89-3, symbol Regulator_Linear:AMS1117-3.3
- added U3: W25Q128JVS, Package_SO:SOIC-8_5.3x5.3mm_P1.27mm, symbol Memory_Flash:W25Q128JVS
Connections:
- new net: R2.1, U1.37 (GPIO25)
- new net: D1.2 (A), R2.2
- new net: C4.1, J1.1 (VBUS), U2.3 (VI)
- new net: R3.1, U1.52 (USB_DP)
- new net: L1.1, U1.48 (VREG_LX)
- new net: R4.1, U1.51 (USB_DM)
- new net: C1.1, R1.2, U1.46 (VREG_AVDD)
- new net 1v1: C3.1, C6.1, C7.1, C8.1, L1.2, U1.23 (DVDD), U1.39 (DVDD), U1.50 (VREG_FB), U1.6 (DVDD)
- new net 3v3: C10.1, C11.1, C12.1, C13.1, C14.1, C15.1, C16.1, C17.1, C2.1, C5.1, C9.1, R1.1, U1.1 (IOVDD), U1.11 (IOVDD), U1.20 (IOVDD), U1.30 (IOVDD), U1.38 (IOVDD), U1.44 (ADC_AVDD), U1.45 (IOVDD), U1.49 (VREG_VIN), U1.53 (USB_OTP_VDD), U1.54 (QSPI_IOVDD), U2.2 (VO)
- new net GND: C1.2, C10.2, C11.2, C12.2, C13.2, C14.2, C15.2, C16.2, C17.2, C2.2, C3.2, C4.2, C5.2, C6.2, C7.2, C8.2, C9.2, D1.1 (K), J1.4 (GND), J1.5 (Shield), U1.47 (VREG_PGND), U1.61 (GND), U2.1 (GND)
- new net QSPI_SCLK: U1.56 (QSPI_SCLK), U3.6 (CLK)
- new net QSPI_SD0: U1.57 (QSPI_SD0), U3.5 (DI/IO_{0})
- new net QSPI_SD1: U1.59 (QSPI_SD1), U3.2 (DO/IO_{1})
- new net QSPI_SD2: U1.58 (QSPI_SD2), U3.3 (~{WP}/IO_{2})
- new net QSPI_SD3: U1.55 (QSPI_SD3), U3.7 (~{HOLD}/~{RESET}/IO_{3})
- new net QSPI_SS: U1.60 (QSPI_SS), U3.1 (~{CS})
- new net RUN: U1.26 (RUN)
- new net SWCLK: U1.24 (SWCLK)
- new net SWDIO: U1.25 (SWDIO)
- new net USB_DM: J1.2 (D-), R4.2
- new net USB_DP: J1.3 (D+), R3.2
- new net XIN: U1.21 (XIN)
- new net XOUT: U1.22 (XOUT)

Commit message: pcb
Parts:
- added C18, C19: 15p, symbol Device:C
- added R5, R6, R7: 1k, symbol Device:R
- added SW1, SW2: SW_Push, symbol Switch:SW_Push
- added Y1: Crystal_GND24, symbol Device:Crystal_GND24
Connections:
- net RUN is gone; now on net 3v3: U1.26 (RUN)
- net 3v3: now also U3.8 (VCC)
- net GND: now also U3.4 (GND), C18.2, C19.2, SW1.1, SW2.2, Y1.2, Y1.4
- net QSPI_SS: now also R6.2
- net XIN: now also C19.1, Y1.1
- net XOUT: now also R5.2
- net at U1.32 (GPIO20): now also R7.1
- new net: C18.1, R5.1, Y1.3
- new net: R7.2, SW2.1
- new net: R6.1, SW1.2
Other:
- moved on the sheet: U3

Commit message: sch + pcb
Parts:
- added D2: ESDS314DBVR, user_imported_devices:ESDS314BVR_SOT95P280X145-5N, symbol user_imported:ESDS314DBVR
- C1, C10, C11, C12, C13, C14, C15, C16, C17, C18, C19, C2, C3, C6, C7, C8, C9: footprint (none) -> Capacitor_SMD:C_0402_1005Metric
- C4, C5: footprint (none) -> Capacitor_SMD:C_0805_2012Metric
- D1: footprint (none) -> LED_SMD:LED_0402_1005Metric
- J1: footprint (none) -> user_imported_devices:USBPCB
- L1: footprint (none) -> Inductor_SMD:L_0402_1005Metric
- R1, R3, R4, R5, R6, R7: footprint (none) -> Resistor_SMD:R_0402_1005Metric
- R2: value 33 -> 1k; footprint (none) -> Resistor_SMD:R_0402_1005Metric
- SW1, SW2: footprint (none) -> Button_Switch_SMD:SW_SPST_PTS810
- Y1: footprint (none) -> Crystal:Crystal_SMD_3225-4Pin_3.2x2.5mm
Connections:
- net USB_DM: now also D2.3 (I/O2)
- net USB_DP: now also D2.1 (I/O1)
- net at R2.1: now also U1.12 (GPIO8); no longer U1.37 (GPIO25)
- net at U1.15 (GPIO11): now also R7.1
- net at U1.32 (GPIO20): no longer R7.1
Other:
- moved on the sheet: C10, C11, C12, C13, C14, C15, C16, C17, C9, D1, R2, R7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

Commit message: pcb
Connections:
- net GND: now also D2.2 (GND)
- net USB_DM: now also D2.1 (I/O1); no longer D2.3 (I/O2)
- net USB_DP: now also D2.3 (I/O2); no longer D2.1 (I/O1)
Changed lines of the file:
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@@
+	(wire
+		(pts
+			(xy 106.68 93.98) (xy 110.49 93.98)
+		)
+		(stroke
+			(width 0)
+			(type default)
+		)
+	)
 	(wire
 		(pts
@@
 	(wire
 		(pts
+			(xy 106.68 88.9) (xy 110.49 88.9)
+		)
+		(stroke
+			(width 0)
+			(type default)
+		)
+	)
+	(wire
+		(pts
 			(xy 143.51 58.42) (xy 156.21 58.42)
 		)
@@
 	(global_label "GND"
 		(shape input)
+		(at 110.49 91.44 180)
+		(fields_autoplaced yes)
+		(effects
+			(font
+				(size 1.27 1.27)
+			)
+			(justify right)
+		)
+		(property "Intersheetrefs" "${INTERSHEET_REFS}"
+			(at 103.6343 91.44 0)
+			(effects
+				(font
+					(size 1.27 1.27)
+				)
+				(justify right)
+				(hide yes)
+			)
+		)
+	)
+	(global_label "GND"
+		(shape input)
 		(at 72.39 106.68 270)
 		(fields_autoplaced yes)
@@
 	(global_label "USB_DP"
 		(shape input)
-		(at 110.49 88.9 180)
-		(fields_autoplaced yes)
-		(effects
-			(font
-				(size 1.27 1.27)
-			)
-			(justify right)
-		)
-		(property "Intersheetrefs" "${INTERSHEET_REFS}"
-			(at 100.1872 88.9 0)
+		(at 106.68 93.98 180)
+		(fields_autoplaced yes)
+		(effects
+			(font
+				(size 1.27 1.27)
+			)
+			(justify right)
+		)
+		(property "Intersheetrefs" "${INTERSHEET_REFS}"
+			(at 96.3772 93.98 0)
 			(effects
 				(font
@@
 	(global_label "USB_DM"
 		(shape input)
-		(at 110.49 93.98 180)
-		(fields_autoplaced yes)
-		(effects
-			(font
-				(size 1.27 1.27)
-			)
-			(justify right)
-		)
-		(property "Intersheetrefs" "${INTERSHEET_REFS}"
-			(at 100.0058 93.98 0)
-			(effects
-				(font
+		(at 106.68 88.9 180)
+		(fields_autoplaced yes)
+		(effects
+			(font
+				(size 1.27 1.27)
+			)
+			(justify right)
+		)
+		(property "Intersheetrefs" "${INTERSHEET_REFS}"
+			(at 96.1958 88.9 0)
+			(effects
+				(font

Commit message: pcb
Connections:
- net at U1.15 (GPIO11): no longer R7.1
- net at U1.37 (GPIO25): now also R7.1
Other:
- moved on the sheet: R7, SW2
Changed lines of the file:
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@@
 	(wire
 		(pts
-			(xy 173.99 27.94) (xy 179.07 27.94)
+			(xy 243.84 129.54) (xy 251.46 129.54)
 		)
 		(stroke
@@
 	(wire
 		(pts
-			(xy 220.98 46.99) (xy 224.79 46.99)
+			(xy 173.99 27.94) (xy 179.07 27.94)
 		)
 		(stroke
@@
 	(wire
 		(pts
-			(xy 243.84 93.98) (xy 251.46 93.98)
+			(xy 220.98 46.99) (xy 224.79 46.99)
 		)
 		(stroke
@@
 	(global_label "GND"
 		(shape input)
-		(at 269.24 93.98 0)
+		(at 269.24 129.54 0)
 		(fields_autoplaced yes)
 		(effects
@@
 		)
 		(property "Intersheetrefs" "${INTERSHEET_REFS}"
-			(at 276.0957 93.98 0)
+			(at 276.0957 129.54 0)
 			(effects
 				(font
@@
 	(symbol
 		(lib_id "Switch:SW_Push")
-		(at 264.16 93.98 0)
+		(at 264.16 129.54 0)
 		(unit 1)
 		(exclude_from_sim no)
@@
 		(dnp no)
 		(property "Reference" "SW2"
-			(at 264.16 96.266 0)
+			(at 264.16 131.826 0)
 			(effects
 				(font
@@
 		)
 		(property "Value" "SW_Push"
-			(at 263.906 98.298 0)
+			(at 263.906 133.858 0)
 			(effects
 				(font
@@
 		)
 		(property "Footprint" "Button_Switch_SMD:SW_SPST_PTS810"
-			(at 264.16 88.9 0)
+			(at 264.16 124.46 0)
 			(effects
 				(font
@@
 		)
 		(property "Datasheet" "~"
-			(at 264.16 88.9 0)
+			(at 264.16 124.46 0)
 			(effects
 				(font
@@
 		)
 		(property "Description" "Push button switch, generic, two pins"
-			(at 264.16 93.98 0)
+			(at 264.16 129.54 0)
 			(effects
 				(font
@@
 	(symbol
 		(lib_id "Device:R")
-		(at 255.27 93.98 90)
+		(at 255.27 129.54 90)
 		(unit 1)
 		(exclude_from_sim no)
@@
 		(dnp no)
 		(property "Reference" "R7"
-			(at 255.27 88.646 90)
+			(at 255.27 124.206 90)
 			(effects
 				(font
@@
 		)
 		(property "Value" "1k"
-			(at 255.27 91.186 90)
+			(at 255.27 126.746 90)
 			(effects
 				(font
@@
 		)
 		(property "Footprint" "Resistor_SMD:R_0402_1005Metric"
-			(at 255.27 95.758 90)
+			(at 255.27 131.318 90)
 			(effects
 				(font
@@
 		)
 		(property "Datasheet" "~"
-			(at 255.27 93.98 0)
+			(at 255.27 129.54 0)
 			(effects
 				(font
@@
 		)
 		(property "Description" "Resistor"
-			(at 255.27 93.98 0)
+			(at 255.27 129.54 0)
 			(effects
 				(font

Commit message: pcb
Parts:
- D1: footprint LED_SMD:LED_0402_1005Metric -> LED_SMD:LED_0402_1005Metric_Pad0.77x0.64mm_HandSolder
- R2, R6, R7: footprint Resistor_SMD:R_0402_1005Metric -> Resistor_SMD:R_0402_1005Metric_Pad0.72x0.64mm_HandSolder
Changed lines of the file:
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@@
 			)
 		)
-		(property "Footprint" "Resistor_SMD:R_0402_1005Metric"
+		(property "Footprint" "Resistor_SMD:R_0402_1005Metric_Pad0.72x0.64mm_HandSolder"
 			(at 255.27 88.138 90)
 			(effects
@@
 			)
 		)
-		(property "Footprint" "LED_SMD:LED_0402_1005Metric"
+		(property "Footprint" "LED_SMD:LED_0402_1005Metric_Pad0.77x0.64mm_HandSolder"
 			(at 262.89 86.36 0)
 			(effects
@@
 			)
 		)
-		(property "Footprint" "Resistor_SMD:R_0402_1005Metric"
+		(property "Footprint" "Resistor_SMD:R_0402_1005Metric_Pad0.72x0.64mm_HandSolder"
 			(at 57.15 77.978 90)
 			(effects
@@
 			)
 		)
-		(property "Footprint" "Resistor_SMD:R_0402_1005Metric"
+		(property "Footprint" "Resistor_SMD:R_0402_1005Metric_Pad0.72x0.64mm_HandSolder"
 			(at 255.27 131.318 90)
 			(effects

Commit message: PCB
Parts:
- L1: footprint Inductor_SMD:L_0402_1005Metric -> Inductor_SMD:L_0805_2012Metric
Changed lines of the file:
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@@
 			)
 		)
-		(property "Footprint" "Inductor_SMD:L_0402_1005Metric"
+		(property "Footprint" "Inductor_SMD:L_0805_2012Metric"
 			(at 156.21 62.23 0)
 			(effects
